Commit message: working simplified arm

File: install/my_robot_controller/share/my_robot_controller/description/robot.urdf.xacro (robot description, xacro)
@@ -29,14 +29,14 @@
   <link name="chassis">
     <visual>
-      <origin xyz="0.1 0 0.075"/>
-      <geometry><box size="0.3 0.3 0.15"/></geometry>
+      <origin xyz="0.1 0 0.025"/>
+      <geometry><box size="0.3 0.3 0.05"/></geometry>
       <material name="blue"/>
     </visual>
     <collision>
-      <origin xyz="0.1 0 0.075"/>
-      <geometry><box size="0.3 0.3 0.15"/></geometry>
+      <origin xyz="0.1 0 0.025"/>
+      <geometry><box size="0.3 0.3 0.05"/></geometry>
     </collision>
-    <xacro:inertial_box mass="0.5" x="0.3" y="0.3" z="0.15">
-        <origin xyz="0.1 0 0.075" rpy="0 0 0"/>
+    <xacro:inertial_box mass="0.5" x="0.3" y="0.3" z="0.05">
+        <origin xyz="0.1 0 0.005" rpy="0 0 0"/>
     </xacro:inertial_box>
   </link>
@@ -65,4 +65,46 @@
   <xacro:wheel prefix="rear_left" x_reflect="-1" y_reflect="1" />
   <xacro:wheel prefix="rear_right" x_reflect="-1" y_reflect="-1" />
+  <link name="arm_1_link">
+    <visual>
+      <origin xyz="0 0 0.1" rpy="0 0 0"/>
+      <geometry><box size="0.05 0.05 0.2"/></geometry>
+      <material name="orange"><color rgba="1 0.5 0 1"/></material>
+    </visual>
+    <collision>
+      <origin xyz="0 0 0.1" rpy="0 0 0"/>
+      <geometry><box size="0.05 0.05 0.2"/></geometry>
+    </collision>
+    <xacro:inertial_box mass="0.1" x="0.05" y="0.05" z="0.2">
+      <origin xyz="0 0 0.1" rpy="0 0 0"/>
+    </xacro:inertial_box>
+  </link>
+  <joint name="shoulder_joint" type="revolute">
+    <parent link="chassis"/>
+    <child link="arm_1_link"/>
+    <origin xyz="0.1 0 0.05" rpy="0 0 0"/>
+    <axis xyz="0 1 0"/> <limit lower="-1.57" upper="1.57" effort="10" velocity="1"/>
+    <dynamics damping="0.1" friction="0.1"/>
+  </joint>
+  <link name="arm_2_link">
+    <visual>
+      <origin xyz="0 0 0.1" rpy="0 0 0"/>
+      <geometry><box size="0.04 0.04 0.2"/></geometry>
+      <material name="orange"/>
+    </visual>
+    <collision>
+      <origin xyz="0 0 0.1" rpy="0 0 0"/>
+      <geometry><box size="0.04 0.04 0.2"/></geometry>
+    </collision>
+    <xacro:inertial_box mass="0.1" x="0.04" y="0.04" z="0.2">
+      <origin xyz="0 0 0.1" rpy="0 0 0"/>
+    </xacro:inertial_box>
+  </link>
+  <joint name="elbow_joint" type="revolute">
+    <parent link="arm_1_link"/>
+    <child link="arm_2_link"/>
+    <origin xyz="0 0 0.2" rpy="0 0 0"/> <axis xyz="0 1 0"/>
+    <limit lower="-2.5" upper="2.5" effort="10" velocity="1"/>
+    <dynamics damping="0.1" friction="0.1"/>
+  </joint>
   <ros2_control name="GazeboSystem" type="system">
     <hardware>
@@ -79,4 +121,14 @@
       </joint>
     </xacro:macro>
+    <joint name="shoulder_joint">
+        <command_interface name="position"/>
+        <state_interface name="position"/>
+        <state_interface name="velocity"/>
+    </joint>
+    <joint name="elbow_joint">
+        <command_interface name="position"/>
+        <state_interface name="position"/>
+        <state_interface name="velocity"/>
+    </joint>
     <xacro:control_joint name="front_left_joint"/>
     <xacro:control_joint name="front_right_joint"/>

Commit message: working map and resized robot

File: install/my_robot_controller/share/my_robot_controller/description/robot.urdf.xacro (robot description, xacro)
@@ -25,18 +25,18 @@
     <parent link="base_link"/>
     <child link="chassis"/>
-    <origin xyz="-0.1 0 0"/>
+    <origin xyz="-0.3 0 0"/>
   </joint>
   <link name="chassis">
     <visual>
-      <origin xyz="0.1 0 0.025"/>
-      <geometry><box size="0.3 0.3 0.05"/></geometry>
+      <origin xyz="0.3 0 0.075"/>
+      <geometry><box size="0.9 0.9 0.15"/></geometry>
       <material name="blue"/>
     </visual>
     <collision>
-      <origin xyz="0.1 0 0.025"/>
-      <geometry><box size="0.3 0.3 0.05"/></geometry>
+      <origin xyz="0.3 0 0.075"/>
+      <geometry><box size="0.9 0.9 0.15"/></geometry>
     </collision>
-    <xacro:inertial_box mass="0.5" x="0.3" y="0.3" z="0.05">
-        <origin xyz="0.1 0 0.005" rpy="0 0 0"/>
+    <xacro:inertial_box mass="0.5" x="0.9" y="0.9" z="0.15">
+        <origin xyz="0.3 0 0.015" rpy="0 0 0"/>
     </xacro:inertial_box>
   </link>
@@ -44,11 +44,11 @@
     <link name="${prefix}_link">
       <visual>
-        <geometry><cylinder radius="0.05" length="0.04"/></geometry>
+        <geometry><cylinder radius="0.15" length="0.12"/></geometry>
         <material name="black"/>
       </visual>
       <collision>
-        <geometry><cylinder radius="0.05" length="0.04"/></geometry>
+        <geometry><cylinder radius="0.15" length="0.12"/></geometry>
       </collision>
-      <xacro:inertial_cylinder mass="0.1" length="0.04" radius="0.05">
+      <xacro:inertial_cylinder mass="0.1" length="0.12" radius="0.15">
         <origin xyz="0 0 0" rpy="0 0 0"/>
       </xacro:inertial_cylinder>
@@ -57,5 +57,5 @@
       <parent link="base_link"/>
       <child link="${prefix}_link"/>
-      <origin xyz="${x_reflect*0.1} ${y_reflect*0.175} 0" rpy="-1.57 0 0"/>
+      <origin xyz="${x_reflect*0.3} ${y_reflect*0.525} 0" rpy="-1.57 0 0"/>
       <axis xyz="0 0 1"/>
     </joint>
@@ -67,14 +67,14 @@
   <link name="arm_1_link">
     <visual>
-      <origin xyz="0 0 0.1" rpy="0 0 0"/>
-      <geometry><box size="0.05 0.05 0.2"/></geometry>
+      <origin xyz="0 0 0.3" rpy="0 0 0"/>
+      <geometry><box size="0.15 0.15 0.6"/></geometry>
       <material name="orange"><color rgba="1 0.5 0 1"/></material>
     </visual>
     <collision>
-      <origin xyz="0 0 0.1" rpy="0 0 0"/>
-      <geometry><box size="0.05 0.05 0.2"/></geometry>
+      <origin xyz="0 0 0.3" rpy="0 0 0"/>
+      <geometry><box size="0.15 0.15 0.6"/></geometry>
     </collision>
-    <xacro:inertial_box mass="0.1" x="0.05" y="0.05" z="0.2">
-      <origin xyz="0 0 0.1" rpy="0 0 0"/>
+    <xacro:inertial_box mass="0.1" x="0.15" y="0.15" z="0.6">
+      <origin xyz="0 0 0.3" rpy="0 0 0"/>
     </xacro:inertial_box>
   </link>
@@ -82,5 +82,5 @@
     <parent link="chassis"/>
     <child link="arm_1_link"/>
-    <origin xyz="0.1 0 0.05" rpy="0 0 0"/>
+    <origin xyz="0.3 0 0.15" rpy="0 0 0"/>
     <axis xyz="0 1 0"/> <limit lower="-1.57" upper="1.57" effort="10" velocity="1"/>
     <dynamics damping="0.1" friction="0.1"/>
@@ -88,14 +88,14 @@
   <link name="arm_2_link">
     <visual>
-      <origin xyz="0 0 0.1" rpy="0 0 0"/>
-      <geometry><box size="0.04 0.04 0.2"/></geometry>
+      <origin xyz="0 0 0.3" rpy="0 0 0"/>
+      <geometry><box size="0.12 0.12 0.6"/></geometry>
       <material name="orange"/>
     </visual>
     <collision>
-      <origin xyz="0 0 0.1" rpy="0 0 0"/>
-      <geometry><box size="0.04 0.04 0.2"/></geometry>
+      <origin xyz="0 0 0.3" rpy="0 0 0"/>
+      <geometry><box size="0.12 0.12 0.6"/></geometry>
     </collision>
-    <xacro:inertial_box mass="0.1" x="0.04" y="0.04" z="0.2">
-      <origin xyz="0 0 0.1" rpy="0 0 0"/>
+    <xacro:inertial_box mass="0.1" x="0.12" y="0.12" z="0.6">
+      <origin xyz="0 0 0.3" rpy="0 0 0"/>
     </xacro:inertial_box>
   </link>
@@ -103,5 +103,5 @@
     <parent link="arm_1_link"/>
     <child link="arm_2_link"/>
-    <origin xyz="0 0 0.2" rpy="0 0 0"/> <axis xyz="0 1 0"/>
+    <origin xyz="0 0 0.6" rpy="0 0 0"/> <axis xyz="0 1 0"/>
     <limit lower="-2.5" upper="2.5" effort="10" velocity="1"/>
     <dynamics damping="0.1" friction="0.1"/>

Commit message: potential grip open and closed

File: install/my_robot_controller/share/my_robot_controller/description/robot.urdf.xacro (robot description, xacro)
@@ -19,6 +19,15 @@
     </inertial>
   </xacro:macro>
+  <!-- MACRO POUR LES CONTROLES - UTILISER VELOCITY -->
+  <xacro:macro name="control_joint" params="name">
+    <joint name="${name}">
+      <command_interface name="velocity"/>
+      <state_interface name="position"/>
+      <state_interface name="velocity"/>
+    </joint>
+  </xacro:macro>
   <material name="blue"><color rgba="0 0 0.8 1"/></material>
   <material name="black"><color rgba="0 0 0 1"/></material>
+  <material name="orange"><color rgba="1 0.5 0 1"/></material>
   <link name="base_link"></link>
   <joint name="chassis_joint" type="fixed">
@@ -69,5 +78,5 @@
       <origin xyz="0 0 0.3" rpy="0 0 0"/>
       <geometry><box size="0.15 0.15 0.6"/></geometry>
-      <material name="orange"><color rgba="1 0.5 0 1"/></material>
+      <material name="orange"/>
     </visual>
     <collision>
@@ -83,5 +92,6 @@
     <child link="arm_1_link"/>
     <origin xyz="0.3 0 0.15" rpy="0 0 0"/>
-    <axis xyz="0 1 0"/> <limit lower="-1.57" upper="1.57" effort="10" velocity="1"/>
+    <axis xyz="0 1 0"/>
+    <limit lower="-1.57" upper="1.57" effort="10" velocity="1"/>
     <dynamics damping="0.1" friction="0.1"/>
   </joint>
@@ -103,7 +113,74 @@
     <parent link="arm_1_link"/>
     <child link="arm_2_link"/>
-    <origin xyz="0 0 0.6" rpy="0 0 0"/> <axis xyz="0 1 0"/>
+    <origin xyz="0 0 0.6" rpy="0 0 0"/>
+    <axis xyz="0 1 0"/>
     <limit lower="-2.5" upper="2.5" effort="10" velocity="1"/>
     <dynamics damping="0.1" friction="0.1"/>
+  </joint>
+  <!-- PINCE - Base de la pince (augmentée aussi) -->
+  <link name="gripper_base_link">
+    <visual>
+      <origin xyz="0 0 0" rpy="0 0 0"/>
+      <geometry><box size="0.3 0.24 0.15"/></geometry>
+      <material name="black"/>
+    </visual>
+    <collision>
+      <origin xyz="0 0 0" rpy="0 0 0"/>
+      <geometry><box size="0.3 0.24 0.15"/></geometry>
+    </collision>
+    <xacro:inertial_box mass="0.15" x="0.3" y="0.24" z="0.15">
+      <origin xyz="0 0 0" rpy="0 0 0"/>
+    </xacro:inertial_box>
+  </link>
+  <joint name="gripper_base_joint" type="fixed">
+    <parent link="arm_2_link"/>
+    <child link="gripper_base_link"/>
+    <origin xyz="0 0 0.6" rpy="0 0 0"/>
+  </joint>
+  <!-- DOIGT GAUCHE (plus mince, plus long) -->
+  <link name="gripper_left_link">
+    <visual>
+      <origin xyz="-0.15 0.15 0.12" rpy="0 0 0"/>
+      <geometry><box size="0.06 0.05 0.36"/></geometry>
+      <material name="black"/>
+    </visual>
+    <collision>
+      <origin xyz="-0.15 0.15 0.12" rpy="0 0 0"/>
+      <geometry><box size="0.06 0.05 0.36"/></geometry>
+    </collision>
+    <xacro:inertial_box mass="0.10" x="0.06" y="0.05" z="0.36">
+      <origin xyz="-0.15 0.15 0.12" rpy="0 0 0"/>
+    </xacro:inertial_box>
+  </link>
+  <joint name="gripper_left_joint" type="prismatic">
+    <parent link="gripper_base_link"/>
+    <child link="gripper_left_link"/>
+    <origin xyz="0 0 0" rpy="0 0 0"/>
+    <axis xyz="1 0 0"/>
+    <limit lower="-0.60" upper="0.0" effort="300" velocity="0.5"/>
+    <dynamics damping="0.5" friction="0.5"/>
+  </joint>
+  <!-- DOIGT DROIT (plus mince, plus long) -->
+  <link name="gripper_right_link">
+    <visual>
+      <origin xyz="0.15 0.15 0.12" rpy="0 0 0"/>
+      <geometry><box size="0.06 0.05 0.36"/></geometry>
+      <material name="black"/>
+    </visual>
+    <collision>
+      <origin xyz="0.15 0.15 0.12" rpy="0 0 0"/>
+      <geometry><box size="0.06 0.05 0.36"/></geometry>
+    </collision>
+    <xacro:inertial_box mass="0.10" x="0.06" y="0.05" z="0.36">
+      <origin xyz="0.15 0.15 0.12" rpy="0 0 0"/>
+    </xacro:inertial_box>
+  </link>
+  <joint name="gripper_right_joint" type="prismatic">
+    <parent link="gripper_base_link"/>
+    <child link="gripper_right_link"/>
+    <origin xyz="0 0 0" rpy="0 0 0"/>
+    <axis xyz="-1 0 0"/>
+    <limit lower="-0.60" upper="0.0" effort="300" velocity="0.5"/>
+    <dynamics damping="0.5" friction="0.5"/>
   </joint>
   <ros2_control name="GazeboSystem" type="system">
@@ -111,14 +188,4 @@
       <plugin>gazebo_ros2_control/GazeboSystem</plugin>
     </hardware>
-    <xacro:macro name="control_joint" params="name">
-      <joint name="${name}">
-        <command_interface name="velocity">
-          <param name="min">-10</param>
-          <param name="max">10</param>
-        </command_interface>
-        <state_interface name="position"/>
-        <state_interface name="velocity"/>
-      </joint>
-    </xacro:macro>
     <joint name="shoulder_joint">
         <command_interface name="position"/>
@@ -127,4 +194,14 @@
     </joint>
     <joint name="elbow_joint">
+        <command_interface name="position"/>
+        <state_interface name="position"/>
+        <state_interface name="velocity"/>
+    </joint>
+    <joint name="gripper_left_joint">
+        <command_interface name="position"/>
+        <state_interface name="position"/>
+        <state_interface name="velocity"/>
+    </joint>
+    <joint name="gripper_right_joint">
         <command_interface name="position"/>
         <state_interface name="position"/>

Commit message: potential grip open and closed rotated

File: install/my_robot_controller/share/my_robot_controller/description/robot.urdf.xacro (robot description, xacro)
@@ -19,15 +19,6 @@
     </inertial>
   </xacro:macro>
-  <!-- MACRO POUR LES CONTROLES - UTILISER VELOCITY -->
-  <xacro:macro name="control_joint" params="name">
-    <joint name="${name}">
-      <command_interface name="velocity"/>
-      <state_interface name="position"/>
-      <state_interface name="velocity"/>
-    </joint>
-  </xacro:macro>
   <material name="blue"><color rgba="0 0 0.8 1"/></material>
   <material name="black"><color rgba="0 0 0 1"/></material>
-  <material name="orange"><color rgba="1 0.5 0 1"/></material>
   <link name="base_link"></link>
   <joint name="chassis_joint" type="fixed">
@@ -78,5 +69,5 @@
       <origin xyz="0 0 0.3" rpy="0 0 0"/>
       <geometry><box size="0.15 0.15 0.6"/></geometry>
-      <material name="orange"/>
+      <material name="orange"><color rgba="1 0.5 0 1"/></material>
     </visual>
     <collision>
@@ -92,6 +83,5 @@
     <child link="arm_1_link"/>
     <origin xyz="0.3 0 0.15" rpy="0 0 0"/>
-    <axis xyz="0 1 0"/>
-    <limit lower="-1.57" upper="1.57" effort="10" velocity="1"/>
+    <axis xyz="0 1 0"/> <limit lower="-1.57" upper="1.57" effort="10" velocity="1"/>
     <dynamics damping="0.1" friction="0.1"/>
   </joint>
@@ -113,10 +103,24 @@
     <parent link="arm_1_link"/>
     <child link="arm_2_link"/>
-    <origin xyz="0 0 0.6" rpy="0 0 0"/>
-    <axis xyz="0 1 0"/>
+    <origin xyz="0 0 0.6" rpy="0 0 0"/> <axis xyz="0 1 0"/>
     <limit lower="-2.5" upper="2.5" effort="10" velocity="1"/>
     <dynamics damping="0.1" friction="0.1"/>
   </joint>
-  <!-- PINCE - Base de la pince (augmentée aussi) -->
+  <!-- PINCE - Joint de rotation (NEW) -->
+  <joint name="gripper_rotate_joint" type="revolute">
+    <parent link="arm_2_link"/>
+    <child link="gripper_base_link"/>
+    <origin xyz="0 0 0.6" rpy="0 0 0"/>
+    <axis xyz="0 0 1"/>
+    <limit lower="-3.14159" upper="3.14159" effort="50" velocity="1.0"/>
+    <dynamics damping="0.1" friction="0.1"/>
+  </joint>
+  <!-- Supprimer l'ancien gripper_base_joint (fixed) -->
+  <!-- <joint name="gripper_base_joint" type="fixed">
+    <parent link="arm_2_link"/>
+    <child link="gripper_base_link"/>
+    <origin xyz="0 0 0.6" rpy="0 0 0"/>
+  </joint> -->
+  <!-- PINCE - Base de la pince -->
   <link name="gripper_base_link">
     <visual>
@@ -133,9 +137,4 @@
     </xacro:inertial_box>
   </link>
-  <joint name="gripper_base_joint" type="fixed">
-    <parent link="arm_2_link"/>
-    <child link="gripper_base_link"/>
-    <origin xyz="0 0 0.6" rpy="0 0 0"/>
-  </joint>
   <!-- DOIGT GAUCHE (plus mince, plus long) -->
   <link name="gripper_left_link">
@@ -188,4 +187,15 @@
       <plugin>gazebo_ros2_control/GazeboSystem</plugin>
     </hardware>
+    <xacro:macro name="control_joint" params="name">
+      <joint name="${name}">
+        <command_interface name="velocity">
+          <param name="min">-10</param>
+          <param name="max">10</param>
+        </command_interface>
+        <state_interface name="position"/>
+        <state_interface name="velocity"/>
+      </joint>
+    </xacro:macro>
+    <!-- Bras + Rotation Grip (POSITION) -->
     <joint name="shoulder_joint">
         <command_interface name="position"/>
@@ -198,18 +208,25 @@
         <state_interface name="velocity"/>
     </joint>
-    <joint name="gripper_left_joint">
-        <command_interface name="position"/>
-        <state_interface name="position"/>
-        <state_interface name="velocity"/>
-    </joint>
-    <joint name="gripper_right_joint">
-        <command_interface name="position"/>
-        <state_interface name="position"/>
-        <state_interface name="velocity"/>
-    </joint>
+    <joint name="gripper_rotate_joint">
+        <command_interface name="position"/>
+        <state_interface name="position"/>
+        <state_interface name="velocity"/>
+    </joint>
+    <!-- Roues (VELOCITY) -->
     <xacro:control_joint name="front_left_joint"/>
     <xacro:control_joint name="front_right_joint"/>
     <xacro:control_joint name="rear_left_joint"/>
     <xacro:control_joint name="rear_right_joint"/>
+    <!-- Pince - Doigts (POSITION) -->
+    <joint name="gripper_left_joint">
+        <command_interface name="position"/>
+        <state_interface name="position"/>
+        <state_interface name="velocity"/>
+    </joint>
+    <joint name="gripper_right_joint">
+        <command_interface name="position"/>
+        <state_interface name="position"/>
+        <state_interface name="velocity"/>
+    </joint>
   </ros2_control>
   <gazebo>

Commit message: Add build logs and model files for my_robot_controller and stl cube

File: install/my_robot_controller/share/my_robot_controller/description/robot.urdf.xacro (robot description, xacro)
@@ -111,5 +111,5 @@
     <parent link="arm_2_link"/>
     <child link="gripper_base_link"/>
-    <origin xyz="0 0 0.6" rpy="0 0 0"/>
+    <origin xyz="0 0 0.6" rpy="0 0 -1.5708"/>
     <axis xyz="0 0 1"/>
     <limit lower="-3.14159" upper="3.14159" effort="50" velocity="1.0"/>
