Commit message: Add autonomous pick-and-place system with SLAM, Nav2, and action servers
- Add LIDAR sensor (lidar.xacro) for SLAM and navigation
- Create custom actions: PickPlace.action, MoveArm.action
- Configure SLAM Toolbox (slam_params.yaml)
- Configure Nav2 navigation stack (nav2_params.yaml)
- Implement action servers: arm_action_server.py, pick_place_action_server.py
- Implement mission orchestrator for A→B→A autonomous operation
- Add launch files: slam_mapping.launch.py, autonomous_mission.launch.py
- Update package.xml and CMakeLists.txt for dependencies and action generation
- Add comprehensive documentation guides

File: install/my_robot_controller/share/my_robot_controller/description/robot.urdf.xacro (robot description, xacro)
@@ -1,237 +1 @@
-<?xml version="1.0"?>
-<robot xmlns:xacro="http://www.ros.org/wiki/xacro" name="mon_robot">
-  <xacro:macro name="inertial_box" params="mass x y z *origin">
-    <inertial>
-      <xacro:insert_block name="origin"/>
-      <mass value="${mass}" />
-      <inertia ixx="${(1/12) * mass * (y*y+z*z)}" ixy="0.0" ixz="0.0"
-               iyy="${(1/12) * mass * (x*x+z*z)}" iyz="0.0"
-               izz="${(1/12) * mass * (x*x+y*y)}" />
-    </inertial>
-  </xacro:macro>
-  <xacro:macro name="inertial_cylinder" params="mass length radius *origin">
-    <inertial>
-      <xacro:insert_block name="origin"/>
-      <mass value="${mass}" />
-      <inertia ixx="${(1/12) * mass * (3*radius*radius + length*length)}" ixy="0.0" ixz="0.0"
-               iyy="${(1/12) * mass * (3*radius*radius + length*length)}" iyz="0.0"
-               izz="${(1/2) * mass * (radius*radius)}" />
-    </inertial>
-  </xacro:macro>
-  <material name="blue"><color rgba="0 0 0.8 1"/></material>
-  <material name="black"><color rgba="0 0 0 1"/></material>
-  <link name="base_link"></link>
-  <joint name="chassis_joint" type="fixed">
-    <parent link="base_link"/>
-    <child link="chassis"/>
-    <origin xyz="-0.3 0 0"/>
-  </joint>
-  <link name="chassis">
-    <visual>
-      <origin xyz="0.3 0 0.075"/>
-      <geometry><box size="0.9 0.9 0.15"/></geometry>
-      <material name="blue"/>
-    </visual>
-    <collision>
-      <origin xyz="0.3 0 0.075"/>
-      <geometry><box size="0.9 0.9 0.15"/></geometry>
-    </collision>
-    <xacro:inertial_box mass="0.5" x="0.9" y="0.9" z="0.15">
-        <origin xyz="0.3 0 0.015" rpy="0 0 0"/>
-    </xacro:inertial_box>
-  </link>
-  <xacro:macro name="wheel" params="prefix x_reflect y_reflect">
-    <link name="${prefix}_link">
-      <visual>
-        <geometry><cylinder radius="0.15" length="0.12"/></geometry>
-        <material name="black"/>
-      </visual>
-      <collision>
-        <geometry><cylinder radius="0.15" length="0.12"/></geometry>
-      </collision>
-      <xacro:inertial_cylinder mass="0.1" length="0.12" radius="0.15">
-        <origin xyz="0 0 0" rpy="0 0 0"/>
-      </xacro:inertial_cylinder>
-    </link>
-    <joint name="${prefix}_joint" type="continuous">
-      <parent link="base_link"/>
-      <child link="${prefix}_link"/>
-      <origin xyz="${x_reflect*0.3} ${y_reflect*0.525} 0" rpy="-1.57 0 0"/>
-      <axis xyz="0 0 1"/>
-    </joint>
-  </xacro:macro>
-  <xacro:wheel prefix="front_left" x_reflect="1" y_reflect="1" />
-  <xacro:wheel prefix="front_right" x_reflect="1" y_reflect="-1" />
-  <xacro:wheel prefix="rear_left" x_reflect="-1" y_reflect="1" />
-  <xacro:wheel prefix="rear_right" x_reflect="-1" y_reflect="-1" />
-  <link name="arm_1_link">
-    <visual>
-      <origin xyz="0 0 0.3" rpy="0 0 0"/>
-      <geometry><box size="0.15 0.15 0.6"/></geometry>
-      <material name="orange"><color rgba="1 0.5 0 1"/></material>
-    </visual>
-    <collision>
-      <origin xyz="0 0 0.3" rpy="0 0 0"/>
-      <geometry><box size="0.15 0.15 0.6"/></geometry>
-    </collision>
-    <xacro:inertial_box mass="0.1" x="0.15" y="0.15" z="0.6">
-      <origin xyz="0 0 0.3" rpy="0 0 0"/>
-    </xacro:inertial_box>
-  </link>
-  <joint name="shoulder_joint" type="revolute">
-    <parent link="chassis"/>
-    <child link="arm_1_link"/>
-    <origin xyz="0.3 0 0.15" rpy="0 0 0"/>
-    <axis xyz="0 1 0"/> <limit lower="-1.57" upper="1.57" effort="10" velocity="1"/>
-    <dynamics damping="0.1" friction="0.1"/>
-  </joint>
-  <link name="arm_2_link">
-    <visual>
-      <origin xyz="0 0 0.3" rpy="0 0 0"/>
-      <geometry><box size="0.12 0.12 0.6"/></geometry>
-      <material name="orange"/>
-    </visual>
-    <collision>
-      <origin xyz="0 0 0.3" rpy="0 0 0"/>
-      <geometry><box size="0.12 0.12 0.6"/></geometry>
-    </collision>
-    <xacro:inertial_box mass="0.1" x="0.12" y="0.12" z="0.6">
-      <origin xyz="0 0 0.3" rpy="0 0 0"/>
-    </xacro:inertial_box>
-  </link>
-  <joint name="elbow_joint" type="revolute">
-    <parent link="arm_1_link"/>
-    <child link="arm_2_link"/>
-    <origin xyz="0 0 0.6" rpy="0 0 0"/> <axis xyz="0 1 0"/>
-    <limit lower="-2.5" upper="2.5" effort="10" velocity="1"/>
-    <dynamics damping="0.1" friction="0.1"/>
-  </joint>
-  <!-- PINCE - Joint de rotation (NEW) -->
-  <joint name="gripper_rotate_joint" type="revolute">
-    <parent link="arm_2_link"/>
-    <child link="gripper_base_link"/>
-    <origin xyz="0 0 0.6" rpy="0 0 -1.5708"/>
-    <axis xyz="0 0 1"/>
-    <limit lower="-3.14159" upper="3.14159" effort="50" velocity="1.0"/>
-    <dynamics damping="0.1" friction="0.1"/>
-  </joint>
-  <!-- Supprimer l'ancien gripper_base_joint (fixed) -->
-  <!-- <joint name="gripper_base_joint" type="fixed">
-    <parent link="arm_2_link"/>
-    <child link="gripper_base_link"/>
-    <origin xyz="0 0 0.6" rpy="0 0 0"/>
-  </joint> -->
-  <!-- PINCE - Base de la pince -->
-  <link name="gripper_base_link">
-    <visual>
-      <origin xyz="0 0 0" rpy="0 0 0"/>
-      <geometry><box size="0.3 0.24 0.15"/></geometry>
-      <material name="black"/>
-    </visual>
-    <collision>
-      <origin xyz="0 0 0" rpy="0 0 0"/>
-      <geometry><box size="0.3 0.24 0.15"/></geometry>
-    </collision>
-    <xacro:inertial_box mass="0.15" x="0.3" y="0.24" z="0.15">
-      <origin xyz="0 0 0" rpy="0 0 0"/>
-    </xacro:inertial_box>
-  </link>
-  <!-- DOIGT GAUCHE (plus mince, plus long) -->
-  <link name="gripper_left_link">
-    <visual>
-      <origin xyz="-0.15 0.15 0.12" rpy="0 0 0"/>
-      <geometry><box size="0.06 0.05 0.36"/></geometry>
-      <material name="black"/>
-    </visual>
-    <collision>
-      <origin xyz="-0.15 0.15 0.12" rpy="0 0 0"/>
-      <geometry><box size="0.06 0.05 0.36"/></geometry>
-    </collision>
-    <xacro:inertial_box mass="0.10" x="0.06" y="0.05" z="0.36">
-      <origin xyz="-0.15 0.15 0.12" rpy="0 0 0"/>
-    </xacro:inertial_box>
-  </link>
-  <joint name="gripper_left_joint" type="prismatic">
-    <parent link="gripper_base_link"/>
-    <child link="gripper_left_link"/>
-    <origin xyz="0 0 0" rpy="0 0 0"/>
-    <axis xyz="1 0 0"/>
-    <limit lower="-0.60" upper="0.0" effort="300" velocity="0.5"/>
-    <dynamics damping="0.5" friction="0.5"/>
-  </joint>
-  <!-- DOIGT DROIT (plus mince, plus long) -->
-  <link name="gripper_right_link">
-    <visual>
-      <origin xyz="0.15 0.15 0.12" rpy="0 0 0"/>
-      <geometry><box size="0.06 0.05 0.36"/></geometry>
-      <material name="black"/>
-    </visual>
-    <collision>
-      <origin xyz="0.15 0.15 0.12" rpy="0 0 0"/>
-      <geometry><box size="0.06 0.05 0.36"/></geometry>
-    </collision>
-    <xacro:inertial_box mass="0.10" x="0.06" y="0.05" z="0.36">
-      <origin xyz="0.15 0.15 0.12" rpy="0 0 0"/>
-    </xacro:inertial_box>
-  </link>
-  <joint name="gripper_right_joint" type="prismatic">
-    <parent link="gripper_base_link"/>
-    <child link="gripper_right_link"/>
-    <origin xyz="0 0 0" rpy="0 0 0"/>
-    <axis xyz="-1 0 0"/>
-    <limit lower="-0.60" upper="0.0" effort="300" velocity="0.5"/>
-    <dynamics damping="0.5" friction="0.5"/>
-  </joint>
-  <ros2_control name="GazeboSystem" type="system">
-    <hardware>
-      <plugin>gazebo_ros2_control/GazeboSystem</plugin>
-    </hardware>
-    <xacro:macro name="control_joint" params="name">
-      <joint name="${name}">
-        <command_interface name="velocity">
-          <param name="min">-10</param>
-          <param name="max">10</param>
-        </command_interface>
-        <state_interface name="position"/>
-        <state_interface name="velocity"/>
-      </joint>
-    </xacro:macro>
-    <!-- Bras + Rotation Grip (POSITION) -->
-    <joint name="shoulder_joint">
-        <command_interface name="position"/>
-        <state_interface name="position"/>
-        <state_interface name="velocity"/>
-    </joint>
-    <joint name="elbow_joint">
-        <command_interface name="position"/>
-        <state_interface name="position"/>
-        <state_interface name="velocity"/>
-    </joint>
-    <joint name="gripper_rotate_joint">
-        <command_interface name="position"/>
-        <state_interface name="position"/>
-        <state_interface name="velocity"/>
-    </joint>
-    <!-- Roues (VELOCITY) -->
-    <xacro:control_joint name="front_left_joint"/>
-    <xacro:control_joint name="front_right_joint"/>
-    <xacro:control_joint name="rear_left_joint"/>
-    <xacro:control_joint name="rear_right_joint"/>
-    <!-- Pince - Doigts (POSITION) -->
-    <joint name="gripper_left_joint">
-        <command_interface name="position"/>
-        <state_interface name="position"/>
-        <state_interface name="velocity"/>
-    </joint>
-    <joint name="gripper_right_joint">
-        <command_interface name="position"/>
-        <state_interface name="position"/>
-        <state_interface name="velocity"/>
-    </joint>
-  </ros2_control>
-  <gazebo>
-    <plugin name="gazebo_ros2_control" filename="libgazebo_ros2_control.so">
-      <parameters>$(find my_robot_controller)/config/my_controllers.yaml</parameters>
-    </plugin>
-  </gazebo>
-</robot>
+/home/lamiae/ROS2_Project/ROS2_Project/src/my_robot_controller/description/robot.urdf.xacro

File: src/my_robot_controller/description/robot.urdf.xacro (robot description, xacro)
@@ -235,3 +235,5 @@
     </plugin>
   </gazebo>
+  <!-- Include LIDAR sensor -->
+  <xacro:include filename="$(find my_robot_controller)/description/lidar.xacro" />
 </robot>

Commit message: Add SLAM and navigation with pick-and-place action

File: install/my_robot_controller/share/my_robot_controller/description/robot.urdf.xacro (robot description, xacro)
@@ -183,4 +183,58 @@
     <dynamics damping="0.5" friction="0.5"/>
   </joint>
+  <!-- LiDAR Sensor -->
+  <link name="lidar_link">
+    <visual>
+      <origin xyz="0 0 0" rpy="0 0 0"/>
+      <geometry>
+        <cylinder radius="0.05" length="0.04"/>
+      </geometry>
+      <material name="black"/>
+    </visual>
+    <collision>
+      <origin xyz="0 0 0" rpy="0 0 0"/>
+      <geometry>
+        <cylinder radius="0.05" length="0.04"/>
+      </geometry>
+    </collision>
+    <xacro:inertial_cylinder mass="0.1" length="0.04" radius="0.05">
+      <origin xyz="0 0 0" rpy="0 0 0"/>
+    </xacro:inertial_cylinder>
+  </link>
+  <joint name="lidar_joint" type="fixed">
+    <parent link="chassis"/>
+    <child link="lidar_link"/>
+    <origin xyz="0.3 0 0.175" rpy="0 0 0"/>
+  </joint>
+  <!-- Gazebo LiDAR Plugin -->
+  <gazebo reference="lidar_link">
+    <sensor name="lidar" type="ray">
+      <always_on>true</always_on>
+      <visualize>true</visualize>
+      <update_rate>10</update_rate>
+      <ray>
+        <scan>
+          <horizontal>
+            <samples>360</samples>
+            <resolution>1.0</resolution>
+            <min_angle>-3.14159</min_angle>
+            <max_angle>3.14159</max_angle>
+          </horizontal>
+        </scan>
+        <range>
+          <min>0.12</min>
+          <max>10.0</max>
+          <resolution>0.01</resolution>
+        </range>
+      </ray>
+      <plugin name="scan" filename="libgazebo_ros_ray_sensor.so">
+        <ros>
+          <remapping>~/out:=scan</remapping>
+        </ros>
+        <output_type>sensor_msgs/LaserScan</output_type>
+        <frame_name>lidar_link</frame_name>
+      </plugin>
+    </sensor>
+  </gazebo>
   <ros2_control name="GazeboSystem" type="system">
     <hardware>

Commit message: update

File: install/my_robot_controller/share/my_robot_controller/description/robot.urdf.xacro (robot description, xacro)
@@ -21,4 +21,5 @@
   <material name="blue"><color rgba="0 0 0.8 1"/></material>
   <material name="black"><color rgba="0 0 0 1"/></material>
+  <material name="red"><color rgba="1 0 0 1"/></material>
   <link name="base_link"></link>
   <joint name="chassis_joint" type="fixed">
@@ -183,4 +184,61 @@
     <dynamics damping="0.5" friction="0.5"/>
   </joint>
+  <!-- CAMERA POUR SUIVI DE LIGNE -->
+  <link name="camera_link">
+    <visual>
+      <origin xyz="0 0 0" rpy="0 0 0"/>
+      <geometry><box size="0.05 0.05 0.05"/></geometry>
+      <material name="red"/>
+    </visual>
+    <collision>
+      <origin xyz="0 0 0" rpy="0 0 0"/>
+      <geometry><box size="0.05 0.05 0.05"/></geometry>
+    </collision>
+    <xacro:inertial_box mass="0.01" x="0.05" y="0.05" z="0.05">
+      <origin xyz="0 0 0" rpy="0 0 0"/>
+    </xacro:inertial_box>
+  </link>
+  <joint name="camera_joint" type="fixed">
+    <parent link="chassis"/>
+    <child link="camera_link"/>
+    <origin xyz="0.35 0 0.01" rpy="0 1.5708 0"/>
+  </joint>
+  <gazebo reference="camera_link">
+    <sensor name="camera_sensor" type="camera">
+      <pose>0 0 0 0 1.5708 0</pose>
+      <update_rate>30.0</update_rate>
+      <camera name="front_camera">
+        <horizontal_fov>1.3962634</horizontal_fov>
+        <image>
+          <width>640</width>
+          <height>480</height>
+          <format>R8G8B8</format>
+        </image>
+        <clip>
+          <near>0.02</near>
+          <far>300</far>
+        </clip>
+        <noise>
+          <type>gaussian</type>
+          <mean>0.0</mean>
+          <stddev>0.007</stddev>
+        </noise>
+      </camera>
+      <plugin name="camera_controller" filename="libgazebo_ros_camera.so">
+        <alwaysOn>true</alwaysOn>
+        <updateRate>0.0</updateRate>
+        <cameraName>robot_camera</cameraName>
+        <imageTopicName>/camera/image_raw</imageTopicName>
+        <cameraInfoTopicName>/camera/camera_info</cameraInfoTopicName>
+        <frameName>camera_link</frameName>
+        <hackBaseline>0.07</hackBaseline>
+        <distortionK1>0.0</distortionK1>
+        <distortionK2>0.0</distortionK2>
+        <distortionK3>0.0</distortionK3>
+        <distortionT1>0.0</distortionT1>
+        <distortionT2>0.0</distortionT2>
+      </plugin>
+    </sensor>
+  </gazebo>
   <ros2_control name="GazeboSystem" type="system">
     <hardware>

Commit message: update

File: install/my_robot_controller/share/my_robot_controller/description/robot.urdf.xacro (robot description, xacro)
@@ -21,4 +21,11 @@
   <material name="blue"><color rgba="0 0 0.8 1"/></material>
   <material name="black"><color rgba="0 0 0 1"/></material>
+  <!-- Base footprint is on the ground under the robot -->
+  <link name="base_footprint"></link>
+  <joint name="base_joint" type="fixed">
+    <parent link="base_footprint"/>
+    <child link="base_link"/>
+    <origin xyz="0 0 0.15" rpy="0 0 0"/>
+  </joint>
   <link name="base_link"></link>
   <joint name="chassis_joint" type="fixed">
