Commit message: Update EKF and SLAM configurations for improved IMU-fused odometry and TF publishing

File: src/my_robot_controller/description/imu.xacro (robot description, xacro)
@@ -24,9 +24,9 @@
     </inertial>
   </link>
-  <!-- Mount IMU on base_link center -->
+  <!-- Mount IMU at chassis center (aligned with base_link origin) -->
   <joint name="imu_joint" type="fixed">
     <parent link="base_link"/>
     <child link="imu_link"/>
-    <origin xyz="0.3 0 0.15" rpy="0 0 0"/>
+    <origin xyz="0 0 0.16" rpy="0 0 0"/>
   </joint>
   <!-- Gazebo IMU Plugin -->
