Commit message: Add robot URDF with a 2-DOF arm, rotating gripper, 4-wheel drive, LIDAR sensor, and initial Nav2/SLAM configurations.

File: src/my_robot_controller/description/lidar.xacro (robot description, xacro)
@@ -61,5 +61,5 @@
         </ros>
         <output_type>sensor_msgs/LaserScan</output_type>
-        <frame_name>laser_frame</frame_name>
+        <frame_name>base_scan</frame_name>
       </plugin>
     </sensor>

File: src/my_robot_controller/description/robot.urdf.xacro (robot description, xacro)
@@ -300,4 +300,14 @@
     </plugin>
   </gazebo>
+  <!-- Static sensor frame for LIDAR (direct child of base_link for Nav2) -->
+  <link name="base_scan"/>
+  <joint name="base_scan_joint" type="fixed">
+    <parent link="base_link"/>
+    <child link="base_scan"/>
+    <!-- Position: base_link is at chassis origin - 0.3
+         laser_frame is at chassis + 0.3, 0, 0.17
+         So from base_link: 0, 0, 0.17 -->
+    <origin xyz="0.0 0 0.17" rpy="0 0 0"/>
+  </joint>
   <!-- Include LIDAR sensor -->
   <xacro:include filename="$(find my_robot_controller)/description/lidar.xacro" />

Commit message: Fix laser scan frame issue - change frame from base_scan to laser_frame

File: src/my_robot_controller/description/lidar.xacro (robot description, xacro)
@@ -61,5 +61,5 @@
         </ros>
         <output_type>sensor_msgs/LaserScan</output_type>
-        <frame_name>base_scan</frame_name>
+        <frame_name>laser_frame</frame_name>
       </plugin>
     </sensor>

File: src/my_robot_controller/description/robot.urdf.xacro (robot description, xacro)
@@ -300,14 +300,4 @@
     </plugin>
   </gazebo>
-  <!-- Static sensor frame for LIDAR (direct child of base_link for Nav2) -->
-  <link name="base_scan"/>
-  <joint name="base_scan_joint" type="fixed">
-    <parent link="base_link"/>
-    <child link="base_scan"/>
-    <!-- Position: base_link is at chassis origin - 0.3
-         laser_frame is at chassis + 0.3, 0, 0.17
-         So from base_link: 0, 0, 0.17 -->
-    <origin xyz="0.0 0 0.17" rpy="0 0 0"/>
-  </joint>
   <!-- Include LIDAR sensor -->
   <xacro:include filename="$(find my_robot_controller)/description/lidar.xacro" />

Commit message: .

File: src/my_robot_controller/description/lidar.xacro (robot description, xacro)
@@ -26,7 +26,7 @@
   <!-- Mount LIDAR on chassis -->
   <joint name="laser_joint" type="fixed">
-    <parent link="chassis"/>
+    <parent link="base_link"/>
     <child link="laser_frame"/>
-    <origin xyz="0.3 0 0.17" rpy="0 0 0"/>
+    <origin xyz="0 0 0.17" rpy="0 0 0"/>
   </joint>
   <!-- Gazebo LIDAR Plugin - OPTIMISÉ POUR SLAM -->

File: src/my_robot_controller/description/robot.urdf.xacro (robot description, xacro)
@@ -35,11 +35,5 @@
     <color rgba="1.0 0.8 0.0 1"/>
   </material>
-  <link name="base_link"></link>
-  <joint name="chassis_joint" type="fixed">
-    <parent link="base_link"/>
-    <child link="chassis"/>
-    <origin xyz="-0.3 0 0"/>
-  </joint>
-  <link name="chassis">
+  <link name="base_link">
     <visual>
       <origin xyz="0.3 0 0.075"/>
@@ -94,5 +88,5 @@
   </link>
   <joint name="shoulder_joint" type="revolute">
-    <parent link="chassis"/>
+    <parent link="base_link"/>
     <child link="arm_1_link"/>
     <origin xyz="0.3 0 0.15" rpy="0 0 0"/>
@@ -245,5 +239,5 @@
   </ros2_control>
   <!-- Gazebo Material Colors -->
-  <gazebo reference="chassis">
+  <gazebo reference="base_link">
     <material>Gazebo/Blue</material>
   </gazebo>

Commit message: feat: amélioration localisation AMCL avec IMU et configuration skid-steer
- Optimisation paramètres AMCL pour robot 4 roues (alpha1-5)
- Ajout IMU sensor dans robot.urdf.xacro
- Configuration LIDAR optimisée pour SLAM
- Amélioration covariances odométrie pour skid-steer
- Augmentation particules AMCL (2000-8000)
- Paramètres laser model optimisés (z_hit, sigma_hit)
- Update rates améliorés (update_min_d, update_min_a)
- Ajout launch_complete_system.launch.py pour lancement complet

File: src/my_robot_controller/description/lidar.xacro (robot description, xacro)
@@ -24,9 +24,9 @@
     </inertial>
   </link>
-  <!-- Mount LIDAR on chassis -->
+  <!-- Mount LIDAR on base_link for stable localization -->
   <joint name="laser_joint" type="fixed">
-    <parent link="chassis"/>
+    <parent link="base_link"/>
     <child link="laser_frame"/>
-    <origin xyz="0.3 0 0.17" rpy="0 0 0"/>
+    <origin xyz="0.0 0 0.32" rpy="0 0 0"/>
   </joint>
   <!-- Gazebo LIDAR Plugin - OPTIMISÉ POUR SLAM -->
@@ -35,9 +35,9 @@
       <pose>0 0 0 0 0 0</pose>
       <visualize>true</visualize>
-      <update_rate>20</update_rate>
+      <update_rate>10</update_rate>
       <ray>
         <scan>
           <horizontal>
-            <samples>720</samples>
+            <samples>360</samples>
             <resolution>1</resolution>
             <min_angle>-3.14159</min_angle>

Commit message: Fix slam launch and robot description; stabilize mapping

File: src/my_robot_controller/description/lidar.xacro (robot description, xacro)
@@ -28,5 +28,5 @@
     <parent link="base_link"/>
     <child link="laser_frame"/>
-    <origin xyz="0 0 0.17" rpy="0 0 0"/>
+    <origin xyz="0 0 0.2" rpy="0 0 0"/>
   </joint>
   <!-- Gazebo LIDAR Plugin - OPTIMISÉ POUR SLAM -->
@@ -35,5 +35,5 @@
       <pose>0 0 0 0 0 0</pose>
       <visualize>true</visualize>
-      <update_rate>20</update_rate>
+      <update_rate>10</update_rate>
       <ray>
         <scan>

File: src/my_robot_controller/description/robot.urdf.xacro (robot description, xacro)
@@ -35,4 +35,11 @@
     <color rgba="1.0 0.8 0.0 1"/>
   </material>
+  <link name="base_footprint">
+  </link>
+  <joint name="base_joint" type="fixed">
+    <parent link="base_footprint"/>
+    <child link="base_link"/>
+    <origin xyz="0 0 0.15" rpy="0 0 0"/>
+  </joint>
   <link name="base_link">
     <visual>
@@ -58,5 +65,5 @@
         <geometry><cylinder radius="0.15" length="0.12"/></geometry>
       </collision>
-      <xacro:inertial_cylinder mass="0.2" length="0.12" radius="0.15">
+      <xacro:inertial_cylinder mass="1.5" length="0.12" radius="0.15">
         <origin xyz="0 0 0" rpy="0 0 0"/>
       </xacro:inertial_cylinder>
@@ -67,4 +74,5 @@
       <origin xyz="${x_reflect*0.3} ${y_reflect*0.525} 0" rpy="-1.57 0 0"/>
       <axis xyz="0 0 1"/>
+      <limit effort="1000.0" velocity="20.0"/>
     </joint>
   </xacro:macro>
@@ -92,5 +100,5 @@
     <origin xyz="0.3 0 0.15" rpy="0 0 0"/>
     <axis xyz="0 1 0"/> <limit lower="-1.57" upper="1.57" effort="10" velocity="1"/>
-    <dynamics damping="0.1" friction="0.1"/>
+    <dynamics damping="10.0" friction="10.0"/>
   </joint>
   <link name="arm_2_link">
@@ -113,5 +121,5 @@
     <origin xyz="-0.3 0 0.6" rpy="0 0 0"/> <axis xyz="0 1 0"/>
     <limit lower="-2.5" upper="2.5" effort="10" velocity="1"/>
-    <dynamics damping="0.1" friction="0.1"/>
+    <dynamics damping="10.0" friction="10.0"/>
   </joint>
   <!-- PINCE - Joint de rotation (NEW) -->
@@ -244,32 +252,32 @@
   <gazebo reference="front_left_link">
     <material>Gazebo/DarkGrey</material>
-    <mu1>100.0</mu1>
-    <mu2>100.0</mu2>
-    <kp>1000000.0</kp>
-    <kd>100.0</kd>
+    <mu1>0.5</mu1>
+    <mu2>0.5</mu2>
+    <kp>100000.0</kp>
+    <kd>10.0</kd>
     <minDepth>0.001</minDepth>
   </gazebo>
   <gazebo reference="front_right_link">
     <material>Gazebo/DarkGrey</material>
-    <mu1>100.0</mu1>
-    <mu2>100.0</mu2>
-    <kp>1000000.0</kp>
-    <kd>100.0</kd>
+    <mu1>0.5</mu1>
+    <mu2>0.5</mu2>
+    <kp>100000.0</kp>
+    <kd>10.0</kd>
     <minDepth>0.001</minDepth>
   </gazebo>
   <gazebo reference="rear_left_link">
     <material>Gazebo/DarkGrey</material>
-    <mu1>100.0</mu1>
-    <mu2>100.0</mu2>
-    <kp>1000000.0</kp>
-    <kd>100.0</kd>
+    <mu1>0.5</mu1>
+    <mu2>0.5</mu2>
+    <kp>100000.0</kp>
+    <kd>10.0</kd>
     <minDepth>0.001</minDepth>
   </gazebo>
   <gazebo reference="rear_right_link">
     <material>Gazebo/DarkGrey</material>
-    <mu1>100.0</mu1>
-    <mu2>100.0</mu2>
-    <kp>1000000.0</kp>
-    <kd>100.0</kd>
+    <mu1>0.5</mu1>
+    <mu2>0.5</mu2>
+    <kp>100000.0</kp>
+    <kd>10.0</kd>
     <minDepth>0.001</minDepth>
   </gazebo>
@@ -291,4 +299,7 @@
   <gazebo>
     <plugin name="gazebo_ros2_control" filename="libgazebo_ros2_control.so">
+      <ros>
+        <remapping>/diff_cont/cmd_vel_unstamped:=/cmd_vel</remapping>
+      </ros>
       <parameters>$(find my_robot_controller)/config/my_controllers.yaml</parameters>
     </plugin>
@@ -296,5 +307,3 @@
   <!-- Include LIDAR sensor -->
   <xacro:include filename="$(find my_robot_controller)/description/lidar.xacro" />
-  <!-- Include IMU sensor -->
-  <xacro:include filename="$(find my_robot_controller)/description/imu.xacro" />
 </robot>
