Commit message: feat: Add new pickup cubes and static obstacles to the world, and refactor robot URDF materials with Gazebo color assignments.

File: src/my_robot_controller/description/robot.urdf.xacro (robot description, xacro)
@@ -19,6 +19,20 @@
     </inertial>
   </xacro:macro>
-  <material name="blue"><color rgba="0 0 0.8 1"/></material>
-  <material name="black"><color rgba="0 0 0 1"/></material>
+  <!-- Enhanced Material Definitions -->
+  <material name="chassis_blue">
+    <color rgba="0.1 0.3 0.6 1"/>
+  </material>
+  <material name="wheel_dark">
+    <color rgba="0.15 0.15 0.15 1"/>
+  </material>
+  <material name="arm_orange">
+    <color rgba="0.9 0.4 0.1 1"/>
+  </material>
+  <material name="gripper_metal">
+    <color rgba="0.3 0.3 0.35 1"/>
+  </material>
+  <material name="accent_yellow">
+    <color rgba="1.0 0.8 0.0 1"/>
+  </material>
   <link name="base_link"></link>
   <joint name="chassis_joint" type="fixed">
@@ -31,5 +45,5 @@
       <origin xyz="0.3 0 0.075"/>
       <geometry><box size="0.9 0.9 0.15"/></geometry>
-      <material name="blue"/>
+      <material name="chassis_blue"/>
     </visual>
     <collision>
@@ -45,5 +59,5 @@
       <visual>
         <geometry><cylinder radius="0.15" length="0.12"/></geometry>
-        <material name="black"/>
+        <material name="wheel_dark"/>
       </visual>
       <collision>
@@ -69,5 +83,5 @@
       <origin xyz="0 0 0.3" rpy="0 0 0"/>
       <geometry><box size="0.15 0.15 0.6"/></geometry>
-      <material name="orange"><color rgba="1 0.5 0 1"/></material>
+      <material name="arm_orange"/>
     </visual>
     <collision>
@@ -90,5 +104,5 @@
       <origin xyz="0 0 0.3" rpy="0 0 0"/>
       <geometry><box size="0.12 0.12 0.6"/></geometry>
-      <material name="orange"/>
+      <material name="arm_orange"/>
     </visual>
     <collision>
@@ -127,5 +141,5 @@
       <origin xyz="0 0 0" rpy="0 0 0"/>
       <geometry><box size="0.3 0.24 0.15"/></geometry>
-      <material name="black"/>
+      <material name="gripper_metal"/>
     </visual>
     <collision>
@@ -142,5 +156,5 @@
       <origin xyz="-0.15 0.15 0.12" rpy="0 0 0"/>
       <geometry><box size="0.06 0.05 0.36"/></geometry>
-      <material name="black"/>
+      <material name="gripper_metal"/>
     </visual>
     <collision>
@@ -165,5 +179,5 @@
       <origin xyz="0.15 0.15 0.12" rpy="0 0 0"/>
       <geometry><box size="0.06 0.05 0.36"/></geometry>
-      <material name="black"/>
+      <material name="gripper_metal"/>
     </visual>
     <collision>
@@ -230,4 +244,35 @@
     </joint>
   </ros2_control>
+  <!-- Gazebo Material Colors -->
+  <gazebo reference="chassis">
+    <material>Gazebo/Blue</material>
+  </gazebo>
+  <gazebo reference="front_left_link">
+    <material>Gazebo/DarkGrey</material>
+  </gazebo>
+  <gazebo reference="front_right_link">
+    <material>Gazebo/DarkGrey</material>
+  </gazebo>
+  <gazebo reference="rear_left_link">
+    <material>Gazebo/DarkGrey</material>
+  </gazebo>
+  <gazebo reference="rear_right_link">
+    <material>Gazebo/DarkGrey</material>
+  </gazebo>
+  <gazebo reference="arm_1_link">
+    <material>Gazebo/Orange</material>
+  </gazebo>
+  <gazebo reference="arm_2_link">
+    <material>Gazebo/Orange</material>
+  </gazebo>
+  <gazebo reference="gripper_base_link">
+    <material>Gazebo/Grey</material>
+  </gazebo>
+  <gazebo reference="gripper_left_link">
+    <material>Gazebo/Grey</material>
+  </gazebo>
+  <gazebo reference="gripper_right_link">
+    <material>Gazebo/Grey</material>
+  </gazebo>
   <gazebo>
     <plugin name="gazebo_ros2_control" filename="libgazebo_ros2_control.so">

Commit message: fused imu

File: src/my_robot_controller/description/robot.urdf.xacro (robot description, xacro)
@@ -37,14 +37,14 @@
   <link name="base_link">
     <visual>
-      <origin xyz="0.3 0 0.075"/>
+      <origin xyz="0 0 0.075"/>
       <geometry><box size="0.9 0.9 0.15"/></geometry>
       <material name="chassis_blue"/>
     </visual>
     <collision>
-      <origin xyz="0.3 0 0.075"/>
+      <origin xyz="0 0 0.075"/>
       <geometry><box size="0.9 0.9 0.15"/></geometry>
     </collision>
     <xacro:inertial_box mass="5.0" x="0.9" y="0.9" z="0.15">
-        <origin xyz="0.3 0 0.015" rpy="0 0 0"/>
+        <origin xyz="0 0 0.075" rpy="0 0 0"/>
     </xacro:inertial_box>
   </link>
@@ -75,14 +75,14 @@
   <link name="arm_1_link">
     <visual>
-      <origin xyz="0 0 0.3" rpy="0 0 0"/>
+      <origin xyz="-0.3 0 0.3" rpy="0 0 0"/>
       <geometry><box size="0.15 0.15 0.6"/></geometry>
       <material name="arm_orange"/>
     </visual>
     <collision>
-      <origin xyz="0 0 0.3" rpy="0 0 0"/>
+      <origin xyz="-0.3 0 0.3" rpy="0 0 0"/>
       <geometry><box size="0.15 0.15 0.6"/></geometry>
     </collision>
     <xacro:inertial_box mass="0.1" x="0.15" y="0.15" z="0.6">
-      <origin xyz="0 0 0.3" rpy="0 0 0"/>
+      <origin xyz="-0.3 0 0.3" rpy="0 0 0"/>
     </xacro:inertial_box>
   </link>
@@ -111,5 +111,5 @@
     <parent link="arm_1_link"/>
     <child link="arm_2_link"/>
-    <origin xyz="0 0 0.6" rpy="0 0 0"/> <axis xyz="0 1 0"/>
+    <origin xyz="-0.3 0 0.6" rpy="0 0 0"/> <axis xyz="0 1 0"/>
     <limit lower="-2.5" upper="2.5" effort="10" velocity="1"/>
     <dynamics damping="0.1" friction="0.1"/>

Commit message: Add IMU sensor to robot

File: src/my_robot_controller/description/robot.urdf.xacro (robot description, xacro)
@@ -35,4 +35,7 @@
     <color rgba="1.0 0.8 0.0 1"/>
   </material>
+  <material name="mat_light_grey">
+    <color rgba="0.7 0.7 0.7 1"/>
+  </material>
   <link name="base_footprint">
   </link>
@@ -81,4 +84,26 @@
   <xacro:wheel prefix="rear_left" x_reflect="-1" y_reflect="1" />
   <xacro:wheel prefix="rear_right" x_reflect="-1" y_reflect="-1" />
+  <!-- IMU Sensor Link -->
+  <link name="imu_link">
+    <visual>
+      <geometry><cylinder radius="0.03" length="0.02"/></geometry>
+      <origin rpy="0 0 0"/>
+      <material name="mat_light_grey"/>
+    </visual>
+    <collision>
+      <geometry><cylinder radius="0.03" length="0.02"/></geometry>
+    </collision>
+    <inertial>
+      <origin xyz="0 0 0"/>
+      <mass value="0.05"/>
+      <inertia ixx="0.000001" ixy="0.0" ixz="0.0"
+               iyy="0.000001" iyz="0.0" izz="0.000001"/>
+    </inertial>
+  </link>
+  <joint name="imu_joint" type="fixed">
+    <parent link="base_link"/>
+    <child link="imu_link"/>
+    <origin xyz="0 0 0.22"/>
+  </joint>
   <link name="arm_1_link">
     <visual>
@@ -297,4 +322,22 @@
     <material>Gazebo/Grey</material>
   </gazebo>
+  <gazebo reference="imu_link">
+    <material>Gazebo/Grey</material>
+  </gazebo>
+  <!-- IMU Sensor Plugin -->
+  <gazebo reference="imu_link">
+    <sensor name="imu" type="imu">
+      <always_on>true</always_on>
+      <update_rate>100</update_rate>
+      <visualize>true</visualize>
+      <plugin name="imu_plugin" filename="libgazebo_ros_imu_sensor.so">
+        <ros>
+          <remapping>~/out:=imu/data</remapping>
+        </ros>
+        <initial_orientation_as_reference>false</initial_orientation_as_reference>
+        <frame_name>imu_link</frame_name>
+      </plugin>
+    </sensor>
+  </gazebo>
   <gazebo>
     <plugin name="gazebo_ros2_control" filename="libgazebo_ros2_control.so">
