Commit message: working bi-derictionnal movement and camera

File: install/blue_line_follower/share/blue_line_follower/urdf/line_follower_robot.urdf.xacro (robot description, xacro)
@@ -135,4 +135,60 @@
     </sensor>
   </gazebo>
+  <!-- Rear Camera Link -->
+  <link name="rear_camera_link">
+    <visual>
+      <geometry>
+        <box size="0.05 0.1 0.05"/>
+      </geometry>
+      <material name="green">
+        <color rgba="0.2 0.8 0.2 1"/>
+      </material>
+    </visual>
+    <collision>
+      <geometry>
+        <box size="0.05 0.1 0.05"/>
+      </geometry>
+    </collision>
+    <inertial>
+      <mass value="0.1"/>
+      <inertia ixx="0.001" ixy="0.0" ixz="0.0" iyy="0.001" iyz="0.0" izz="0.001"/>
+    </inertial>
+  </link>
+  <joint name="rear_camera_joint" type="fixed">
+    <parent link="base_link"/>
+    <child link="rear_camera_link"/>
+    <origin xyz="${-base_length/2 - 0.025} 0 ${base_height/2 + 0}" rpy="0 0.6 3.14159"/>
+  </joint>
+  <!-- Rear Camera Sensor -->
+  <gazebo reference="rear_camera_link">
+    <sensor type="camera" name="rear_camera">
+      <update_rate>30.0</update_rate>
+      <camera name="rear">
+        <horizontal_fov>1.3962634</horizontal_fov>
+        <image>
+          <width>640</width>
+          <height>480</height>
+          <format>R8G8B8</format>
+        </image>
+        <clip>
+          <near>0.02</near>
+          <far>300</far>
+        </clip>
+        <noise>
+          <type>gaussian</type>
+          <mean>0.0</mean>
+          <stddev>0.007</stddev>
+        </noise>
+      </camera>
+      <plugin name="rear_camera_controller" filename="libgazebo_ros_camera.so">
+        <frame_name>rear_camera_link</frame_name>
+        <ros>
+          <namespace>/</namespace>
+          <remapping>~/image_raw:=rear_camera/image_raw</remapping>
+          <remapping>~/camera_info:=rear_camera/camera_info</remapping>
+        </ros>
+      </plugin>
+    </sensor>
+  </gazebo>
   <!-- Differential Drive Plugin -->
   <gazebo>

Commit message: added obstacle detection

File: install/blue_line_follower/share/blue_line_follower/urdf/line_follower_robot.urdf.xacro (robot description, xacro)
@@ -218,4 +218,140 @@
     </plugin>
   </gazebo>
+  <!-- Front Ultrasonic Sensor Link -->
+  <link name="front_ultrasonic_link">
+    <visual>
+      <geometry>
+        <box size="0.02 0.04 0.02"/>
+      </geometry>
+      <material name="yellow">
+        <color rgba="0.9 0.9 0.2 1"/>
+      </material>
+    </visual>
+    <collision>
+      <geometry>
+        <box size="0.02 0.04 0.02"/>
+      </geometry>
+    </collision>
+    <inertial>
+      <mass value="0.01"/>
+      <inertia ixx="0.0001" ixy="0.0" ixz="0.0" iyy="0.0001" iyz="0.0" izz="0.0001"/>
+    </inertial>
+  </link>
+  <joint name="front_ultrasonic_joint" type="fixed">
+    <parent link="camera_link"/>
+    <child link="front_ultrasonic_link"/>
+    <origin xyz="0.0 0 -0.05" rpy="0 -0.6 0"/>
+  </joint>
+  <!-- Front Ultrasonic Sensor -->
+  <gazebo reference="front_ultrasonic_link">
+    <sensor type="ray" name="front_ultrasonic_sensor">
+      <pose>0 0 0 0 0 0</pose>
+      <visualize>true</visualize>
+      <update_rate>10</update_rate>
+      <ray>
+        <scan>
+          <horizontal>
+            <samples>5</samples>
+            <resolution>1</resolution>
+            <min_angle>-0.12</min_angle>
+            <max_angle>0.12</max_angle>
+          </horizontal>
+          <vertical>
+            <samples>5</samples>
+            <resolution>1</resolution>
+            <min_angle>-0.12</min_angle>
+            <max_angle>0.12</max_angle>
+          </vertical>
+        </scan>
+        <range>
+          <min>0.02</min>
+          <max>2.0</max>
+          <resolution>0.01</resolution>
+        </range>
+        <noise>
+          <type>gaussian</type>
+          <mean>0.0</mean>
+          <stddev>0.01</stddev>
+        </noise>
+      </ray>
+      <plugin name="front_ultrasonic_controller" filename="libgazebo_ros_ray_sensor.so">
+        <ros>
+          <namespace>/</namespace>
+          <remapping>~/out:=front_ultrasonic/range</remapping>
+        </ros>
+        <output_type>sensor_msgs/Range</output_type>
+        <frame_name>front_ultrasonic_link</frame_name>
+        <radiation_type>ultrasound</radiation_type>
+      </plugin>
+    </sensor>
+  </gazebo>
+  <!-- Rear Ultrasonic Sensor Link -->
+  <link name="rear_ultrasonic_link">
+    <visual>
+      <geometry>
+        <box size="0.02 0.04 0.02"/>
+      </geometry>
+      <material name="yellow">
+        <color rgba="0.9 0.9 0.2 1"/>
+      </material>
+    </visual>
+    <collision>
+      <geometry>
+        <box size="0.02 0.04 0.02"/>
+      </geometry>
+    </collision>
+    <inertial>
+      <mass value="0.01"/>
+      <inertia ixx="0.0001" ixy="0.0" ixz="0.0" iyy="0.0001" iyz="0.0" izz="0.0001"/>
+    </inertial>
+  </link>
+  <joint name="rear_ultrasonic_joint" type="fixed">
+    <parent link="rear_camera_link"/>
+    <child link="rear_ultrasonic_link"/>
+    <origin xyz="0.0 0 -0.05" rpy="0 -0.6 0"/>
+  </joint>
+  <!-- Rear Ultrasonic Sensor -->
+  <gazebo reference="rear_ultrasonic_link">
+    <sensor type="ray" name="rear_ultrasonic_sensor">
+      <pose>0 0 0 0 0 0</pose>
+      <visualize>true</visualize>
+      <update_rate>10</update_rate>
+      <ray>
+        <scan>
+          <horizontal>
+            <samples>5</samples>
+            <resolution>1</resolution>
+            <min_angle>-0.12</min_angle>
+            <max_angle>0.12</max_angle>
+          </horizontal>
+          <vertical>
+            <samples>5</samples>
+            <resolution>1</resolution>
+            <min_angle>-0.12</min_angle>
+            <max_angle>0.12</max_angle>
+          </vertical>
+        </scan>
+        <range>
+          <min>0.02</min>
+          <max>2.0</max>
+          <resolution>0.01</resolution>
+        </range>
+        <noise>
+          <type>gaussian</type>
+          <mean>0.0</mean>
+          <stddev>0.01</stddev>
+        </noise>
+      </ray>
+      <plugin name="rear_ultrasonic_controller" filename="libgazebo_ros_ray_sensor.so">
+        <ros>
+          <namespace>/</namespace>
+          <remapping>~/out:=rear_ultrasonic/range</remapping>
+        </ros>
+        <output_type>sensor_msgs/Range</output_type>
+        <frame_name>rear_ultrasonic_link</frame_name>
+        <radiation_type>ultrasound</radiation_type>
+      </plugin>
+    </sensor>
+  </gazebo>
   <!-- Gazebo base_link material -->
   <gazebo reference="base_link">

Commit message: added 3rd camera and centering logic

File: install/blue_line_follower/share/blue_line_follower/urdf/line_follower_robot.urdf.xacro (robot description, xacro)
@@ -191,4 +191,60 @@
     </sensor>
   </gazebo>
+  <!-- Bottom Camera Link (fixed under chassis) -->
+  <link name="bottom_camera_link">
+    <visual>
+      <geometry>
+        <box size="0.05 0.05 0.02"/>
+      </geometry>
+      <material name="yellow">
+        <color rgba="0.8 0.8 0.2 1"/>
+      </material>
+    </visual>
+    <collision>
+      <geometry>
+        <box size="0.05 0.05 0.02"/>
+      </geometry>
+    </collision>
+    <inertial>
+      <mass value="0.05"/>
+      <inertia ixx="0.0001" ixy="0.0" ixz="0.0" iyy="0.0001" iyz="0.0" izz="0.0001"/>
+    </inertial>
+  </link>
+  <joint name="bottom_camera_joint" type="fixed">
+    <parent link="base_link"/>
+    <child link="bottom_camera_link"/>
+    <origin xyz="0 0 ${-base_height/2 }" rpy="0 1.5708 0"/>
+  </joint>
+  <!-- Bottom Camera Sensor -->
+  <gazebo reference="bottom_camera_link">
+    <sensor type="camera" name="bottom_camera">
+      <update_rate>30.0</update_rate>
+      <camera name="bottom">
+        <horizontal_fov>1.3962634</horizontal_fov>
+        <image>
+          <width>640</width>
+          <height>640</height>
+          <format>R8G8B8</format>
+        </image>
+        <clip>
+          <near>0.02</near>
+          <far>2.0</far>
+        </clip>
+        <noise>
+          <type>gaussian</type>
+          <mean>0.0</mean>
+          <stddev>0.007</stddev>
+        </noise>
+      </camera>
+      <plugin name="bottom_camera_controller" filename="libgazebo_ros_camera.so">
+        <frame_name>bottom_camera_link</frame_name>
+        <ros>
+          <namespace>/</namespace>
+          <remapping>~/image_raw:=bottom_camera/image_raw</remapping>
+          <remapping>~/camera_info:=bottom_camera/camera_info</remapping>
+        </ros>
+      </plugin>
+    </sensor>
+  </gazebo>
   <!-- Differential Drive Plugin -->
   <gazebo>

Commit message: working rotation

File: install/blue_line_follower/share/blue_line_follower/urdf/line_follower_robot.urdf.xacro (robot description, xacro)
@@ -247,29 +247,50 @@
     </sensor>
   </gazebo>
-  <!-- Differential Drive Plugin -->
+  <!-- ros2_control -->
+  <ros2_control name="gazebo_ros2_control" type="system">
+    <hardware>
+      <plugin>gazebo_ros2_control/GazeboSystem</plugin>
+    </hardware>
+    <!-- Front Left Wheel Joint -->
+    <joint name="front_left_wheel_joint">
+      <command_interface name="velocity">
+        <param name="min">-10</param>
+        <param name="max">10</param>
+      </command_interface>
+      <state_interface name="position"/>
+      <state_interface name="velocity"/>
+    </joint>
+    <!-- Front Right Wheel Joint -->
+    <joint name="front_right_wheel_joint">
+      <command_interface name="velocity">
+        <param name="min">-10</param>
+        <param name="max">10</param>
+      </command_interface>
+      <state_interface name="position"/>
+      <state_interface name="velocity"/>
+    </joint>
+    <!-- Rear Left Wheel Joint -->
+    <joint name="rear_left_wheel_joint">
+      <command_interface name="velocity">
+        <param name="min">-10</param>
+        <param name="max">10</param>
+      </command_interface>
+      <state_interface name="position"/>
+      <state_interface name="velocity"/>
+    </joint>
+    <!-- Rear Right Wheel Joint -->
+    <joint name="rear_right_wheel_joint">
+      <command_interface name="velocity">
+        <param name="min">-10</param>
+        <param name="max">10</param>
+      </command_interface>
+      <state_interface name="position"/>
+      <state_interface name="velocity"/>
+    </joint>
+  </ros2_control>
+  <!-- Gazebo ros2_control plugin -->
   <gazebo>
-    <plugin name="differential_drive_controller" filename="libgazebo_ros_diff_drive.so">
-      <update_rate>50</update_rate>
-      <!-- Wheels -->
-      <left_joint>front_left_wheel_joint</left_joint>
-      <right_joint>front_right_wheel_joint</right_joint>
-      <!-- Kinematics -->
-      <wheel_separation>${wheel_separation}</wheel_separation>
-      <wheel_diameter>${2*wheel_radius}</wheel_diameter>
-      <!-- Limits -->
-      <max_wheel_torque>50</max_wheel_torque>
-      <max_wheel_acceleration>2.0</max_wheel_acceleration>
-      <!-- Output -->
-      <publish_odom>true</publish_odom>
-      <publish_odom_tf>true</publish_odom_tf>
-      <publish_wheel_tf>false</publish_wheel_tf>
-      <odometry_frame>odom</odometry_frame>
-      <robot_base_frame>base_footprint</robot_base_frame>
-      <!-- Topic -->
-      <ros>
-        <namespace>/</namespace>
-        <remapping>cmd_vel:=cmd_vel</remapping>
-        <remapping>odom:=odom</remapping>
-      </ros>
+    <plugin filename="libgazebo_ros2_control.so" name="gazebo_ros2_control">
+      <parameters>$(find blue_line_follower)/config/controller_config.yaml</parameters>
     </plugin>
   </gazebo>

Commit message: prototype of pusher

File: install/blue_line_follower/share/blue_line_follower/urdf/line_follower_robot.urdf.xacro (robot description, xacro)
@@ -435,3 +435,78 @@
     <material>Gazebo/Blue</material>
   </gazebo>
+  <!-- ===== PUSHER MECHANISM ===== -->
+  <!-- Rail horizontal fixé au-dessus du robot (axe longitudinal) -->
+  <link name="pusher_rail_link">
+    <visual>
+      <geometry>
+        <box size="0.7 0.05 0.03"/>
+      </geometry>
+      <material name="silver">
+        <color rgba="0.7 0.7 0.7 1"/>
+      </material>
+    </visual>
+    <collision>
+      <geometry>
+        <box size="0.7 0.05 0.03"/>
+      </geometry>
+    </collision>
+    <inertial>
+      <mass value="0.3"/>
+      <inertia ixx="0.001" ixy="0.0" ixz="0.0" iyy="0.012" iyz="0.0" izz="0.012"/>
+    </inertial>
+  </link>
+  <joint name="pusher_rail_joint" type="fixed">
+    <parent link="base_link"/>
+    <child link="pusher_rail_link"/>
+    <origin xyz="0 0 ${base_height/2 + 0.25}" rpy="0 0 0"/>
+  </joint>
+  <!-- Prisme pousseur - Se déplace d'arrière vers l'avant -->
+  <link name="pusher_arm_link">
+    <visual>
+      <geometry>
+        <box size="0.15 0.3 0.12"/>
+      </geometry>
+      <material name="orange">
+        <color rgba="1.0 0.5 0.0 1"/>
+      </material>
+    </visual>
+    <collision>
+      <geometry>
+        <box size="0.15 0.3 0.12"/>
+      </geometry>
+    </collision>
+    <inertial>
+      <mass value="0.2"/>
+      <inertia ixx="0.001" ixy="0.0" ixz="0.0" iyy="0.001" iyz="0.0" izz="0.001"/>
+    </inertial>
+  </link>
+  <!-- Joint prismatique - permet au pousseur de glisser d'arrière vers l'avant -->
+  <joint name="pusher_joint" type="prismatic">
+    <parent link="pusher_rail_link"/>
+    <child link="pusher_arm_link"/>
+    <origin xyz="${-base_length/2 + 0.1} 0 -0.075" rpy="0 0 0"/>
+    <axis xyz="1 0 0"/>
+    <limit lower="0.0" upper="0.6" effort="50.0" velocity="0.5"/>
+  </joint>
+  <!-- Add pusher to ros2_control -->
+  <ros2_control name="pusher_control" type="system">
+    <hardware>
+      <plugin>gazebo_ros2_control/GazeboSystem</plugin>
+    </hardware>
+    <joint name="pusher_joint">
+      <command_interface name="position">
+        <param name="min">-0.25</param>
+        <param name="max">0.25</param>
+      </command_interface>
+      <state_interface name="position"/>
+      <state_interface name="velocity"/>
+    </joint>
+  </ros2_control>
+  <!-- Gazebo materials for pusher -->
+  <gazebo reference="pusher_rail_link">
+    <material>Gazebo/White</material>
+  </gazebo>
+  <gazebo reference="pusher_arm_link">
+    <material>Gazebo/Orange</material>
+  </gazebo>
 </robot>

Commit message: adjusted camera for box push

File: install/blue_line_follower/share/blue_line_follower/urdf/line_follower_robot.urdf.xacro (robot description, xacro)
@@ -4,5 +4,5 @@
   <xacro:property name="base_width" value="0.4"/>
   <xacro:property name="base_length" value="0.6"/>
-  <xacro:property name="base_height" value="0.15"/>
+  <xacro:property name="base_height" value="0.25"/>
   <xacro:property name="wheel_radius" value="0.1"/>
   <xacro:property name="wheel_width" value="0.05"/>
@@ -83,5 +83,5 @@
     <visual>
       <geometry>
-        <box size="0.05 0.1 0.05"/>
+        <box size="0.03 0.05 0.03"/>
       </geometry>
       <material name="red">
@@ -91,10 +91,10 @@
     <collision>
       <geometry>
-        <box size="0.05 0.1 0.05"/>
-      </geometry>
-    </collision>
-    <inertial>
-      <mass value="0.1"/>
-      <inertia ixx="0.001" ixy="0.0" ixz="0.0" iyy="0.001" iyz="0.0" izz="0.001"/>
+        <box size="0.03 0.05 0.03"/>
+      </geometry>
+    </collision>
+    <inertial>
+      <mass value="0.05"/>
+      <inertia ixx="0.0001" ixy="0.0" ixz="0.0" iyy="0.0001" iyz="0.0" izz="0.0001"/>
     </inertial>
   </link>
@@ -102,5 +102,5 @@
     <parent link="base_link"/>
     <child link="camera_link"/>
-    <origin xyz="${base_length/2 + 0.025} 0 ${base_height/2 + 0}" rpy="0 0.6 0"/>
+    <origin xyz="${base_length/2 + 0.025} 0 ${-base_height/2 + 0.12}" rpy="0 0.6 0"/>
   </joint>
   <!-- Camera Sensor -->
@@ -139,5 +139,5 @@
     <visual>
       <geometry>
-        <box size="0.05 0.1 0.05"/>
+        <box size="0.03 0.05 0.03"/>
       </geometry>
       <material name="green">
@@ -147,10 +147,10 @@
     <collision>
       <geometry>
-        <box size="0.05 0.1 0.05"/>
-      </geometry>
-    </collision>
-    <inertial>
-      <mass value="0.1"/>
-      <inertia ixx="0.001" ixy="0.0" ixz="0.0" iyy="0.001" iyz="0.0" izz="0.001"/>
+        <box size="0.03 0.05 0.03"/>
+      </geometry>
+    </collision>
+    <inertial>
+      <mass value="0.05"/>
+      <inertia ixx="0.0001" ixy="0.0" ixz="0.0" iyy="0.0001" iyz="0.0" izz="0.0001"/>
     </inertial>
   </link>
@@ -158,5 +158,5 @@
     <parent link="base_link"/>
     <child link="rear_camera_link"/>
-    <origin xyz="${-base_length/2 - 0.025} 0 ${base_height/2 + 0}" rpy="0 0.6 3.14159"/>
+    <origin xyz="${-base_length/2 - 0.025} 0 ${-base_height/2 + 0.12}" rpy="0 0.6 3.14159"/>
   </joint>
   <!-- Rear Camera Sensor -->

Commit message: adjusted world

File: install/blue_line_follower/share/blue_line_follower/urdf/line_follower_robot.urdf.xacro (robot description, xacro)
@@ -102,5 +102,5 @@
     <parent link="base_link"/>
     <child link="camera_link"/>
-    <origin xyz="${base_length/2 + 0.025} 0 ${-base_height/2 + 0.12}" rpy="0 0.6 0"/>
+    <origin xyz="${base_length/2 + 0.025} 0 ${-base_height/2 + 0.18}" rpy="0 0.6 0"/>
   </joint>
   <!-- Camera Sensor -->
@@ -158,5 +158,5 @@
     <parent link="base_link"/>
     <child link="rear_camera_link"/>
-    <origin xyz="${-base_length/2 - 0.025} 0 ${-base_height/2 + 0.12}" rpy="0 0.6 3.14159"/>
+    <origin xyz="${-base_length/2 - 0.025} 0 ${-base_height/2 + 0.18}" rpy="0 0.6 3.14159"/>
   </joint>
   <!-- Rear Camera Sensor -->
@@ -436,34 +436,9 @@
   </gazebo>
   <!-- ===== PUSHER MECHANISM ===== -->
-  <!-- Rail horizontal fixé au-dessus du robot (axe longitudinal) -->
-  <link name="pusher_rail_link">
-    <visual>
-      <geometry>
-        <box size="0.7 0.05 0.03"/>
-      </geometry>
-      <material name="silver">
-        <color rgba="0.7 0.7 0.7 1"/>
-      </material>
-    </visual>
-    <collision>
-      <geometry>
-        <box size="0.7 0.05 0.03"/>
-      </geometry>
-    </collision>
-    <inertial>
-      <mass value="0.3"/>
-      <inertia ixx="0.001" ixy="0.0" ixz="0.0" iyy="0.012" iyz="0.0" izz="0.012"/>
-    </inertial>
-  </link>
-  <joint name="pusher_rail_joint" type="fixed">
-    <parent link="base_link"/>
-    <child link="pusher_rail_link"/>
-    <origin xyz="0 0 ${base_height/2 + 0.25}" rpy="0 0 0"/>
-  </joint>
-  <!-- Prisme pousseur - Se déplace d'arrière vers l'avant -->
+  <!-- Prisme pousseur - Collé au dessus du châssis, se déplace d'arrière vers l'avant -->
   <link name="pusher_arm_link">
     <visual>
       <geometry>
-        <box size="0.15 0.3 0.12"/>
+        <box size="0.12 0.12 0.03"/>
       </geometry>
       <material name="orange">
@@ -473,17 +448,17 @@
     <collision>
       <geometry>
-        <box size="0.15 0.3 0.12"/>
-      </geometry>
-    </collision>
-    <inertial>
-      <mass value="0.2"/>
-      <inertia ixx="0.001" ixy="0.0" ixz="0.0" iyy="0.001" iyz="0.0" izz="0.001"/>
+        <box size="0.12 0.12 0.12"/>
+      </geometry>
+    </collision>
+    <inertial>
+      <mass value="0.08"/>
+      <inertia ixx="0.0005" ixy="0.0" ixz="0.0" iyy="0.0005" iyz="0.0" izz="0.0005"/>
     </inertial>
   </link>
   <!-- Joint prismatique - permet au pousseur de glisser d'arrière vers l'avant -->
   <joint name="pusher_joint" type="prismatic">
-    <parent link="pusher_rail_link"/>
+    <parent link="base_link"/>
     <child link="pusher_arm_link"/>
-    <origin xyz="${-base_length/2 + 0.1} 0 -0.075" rpy="0 0 0"/>
+    <origin xyz="${-base_length/2 + 0.06} 0 ${base_height/2 + 0.015}" rpy="0 0 0"/>
     <axis xyz="1 0 0"/>
     <limit lower="0.0" upper="0.6" effort="50.0" velocity="0.5"/>
@@ -504,7 +479,4 @@
   </ros2_control>
   <!-- Gazebo materials for pusher -->
-  <gazebo reference="pusher_rail_link">
-    <material>Gazebo/White</material>
-  </gazebo>
   <gazebo reference="pusher_arm_link">
     <material>Gazebo/Orange</material>
